File: uRinks_v2.0.sch (EAGLE design)
At the start: 136 parts, among them IC1 LM1117-3.3, IC2 STM32F405RGT6, IC3 LM4040B10, IC4 4051PW, IC5 MCP6002, IC6 WM8731, IC7 MCP6004-I_ST, IC8 TL072, J1 WQP-PJ301M-12_JACK, J10 WQP-PJ301M-12_JACK, J2 WQP-PJ301M-12_JACK, J3 WQP-PJ301M-12_JACK, J4 WQP-PJ301M-12_JACK, J5 WQP-PJ301M-12_JACK, J6 WQP-PJ301M-12_JACK, J7 WQP-PJ301M-12_JACK, J8 WQP-PJ301M-12_JACK, J9 WQP-PJ301M-12_JACK, Q1 8MHz, Q2 MMBT3904, Q3 12.288MHz

Commit message: uRinks files
Other:
- note added: "Codex-Modulex"
- note added: "Original design by: Olivier Gillet of Mutable Instruments"
- note added: "info@codex-modulex.com"
- note removed: "Olivier Gillet"
- note removed: "ol.gillet@gmail.com"
